File: Tareas/PRACTICAS DE KICAD/TAREA 2 USB ISOLATED/TAREA_2/TAREA_2.kicad_pcb (KiCad board)
At the start: 2 copper layers, 46.4 x 24.1 mm, 16 parts, among them CN1 USB-B-Female-90, U1 ADUM3166BRSZ, U2 B0503S-1WR3_C5444000, X1 3N24000G33YC

Commit message: changes
Parts:
- added U3: TVSS5VCES-02GP-J_C7473318, EasyEDA:SOD-523_L1.2-W0.8-LS1.6-BI, F.Cu at (169.5, 108.6)
- added U4: TVSS5VCES-02GP-J_C7473318, EasyEDA:SOD-523_L1.2-W0.8-LS1.6-BI, F.Cu at (170.8, 111.0)
- added U5: TVSS5VCES-02GP-J_C7473318, EasyEDA:SOD-523_L1.2-W0.8-LS1.6-BI, F.Cu at (190.9, 108.8)
- added U6: TVSS5VCES-02GP-J_C7473318, EasyEDA:SOD-523_L1.2-W0.8-LS1.6-BI, F.Cu at (190.0, 111.0)
Routing:
- net GND2: vias 36 -> 39
- net GND: vias 32 -> 39
- net (no net): vias 0 -> 4
Other:
- board size 46.4 x 24.1 mm -> 46.4 x 24.8 mm
